File: Tiskana_plocica_za_lego_auto/Tiskana_plocica_za_lego_auto.kicad_sch (KiCad schematic)
At the start: 44 parts, among them J1 Conn_01x16_Pin, J2 Conn_01x20_Pin, J3 Screw_Terminal_01x02, J4 Screw_Terminal_01x02, J6 Screw_Terminal_01x02, J7 Screw_Terminal_01x02, J8 Screw_Terminal_01x04, M1 Motor_DC, M2 Motor_Servo, U1 L298N, U2 LM78M05_TO220, U4 LM2596S-5

Commit message: schema
Parts:
- removed BT1: Battery_Cell, symbol Device:Battery_Cell
- removed D10, D11, D14, D15: D_Zener_Filled, symbol Device:D_Zener_Filled
- removed J1: Conn_01x16_Pin, symbol Connector:Conn_01x16_Pin
- removed J2: Conn_01x20_Pin, symbol Connector:Conn_01x20_Pin
- removed J3, J4, J7: Screw_Terminal_01x02, symbol Connector:Screw_Terminal_01x02
- removed J8: Screw_Terminal_01x04, symbol Connector:Screw_Terminal_01x04
- removed M1: Motor_DC, symbol Motor:Motor_DC
- removed M2: Motor_Servo, symbol Motor:Motor_Servo
- removed R3, R4: R, symbol Device:R
- added H1, H2, H3, H4: MountingHole, MountingHole:MountingHole_8.4mm_M8, symbol Mechanical:MountingHole
- added J1: Conn_01x02_Socket, symbol Connector:Conn_01x02_Socket
- added J2: Conn_01x20_Socket, Connector_PinHeader_2.54mm:PinHeader_1x20_P2.54mm_Vertical_SMD_Pin1Left, symbol Connector:Conn_01x20_Socket
- added J7: Conn_01x20_Socket, Connector_PinSocket_2.54mm:PinSocket_1x20_P2.54mm_Vertical_SMD_Pin1Right, symbol Connector:Conn_01x20_Socket
- added J8: Conn_01x03_Pin, Connector_PinHeader_2.54mm:PinHeader_1x03_P2.54mm_Vertical_SMD_Pin1Right, symbol Connector:Conn_01x03_Pin
- added Q1: IRLZ44N, Package_TO_SOT_THT:TO-220-3_Vertical, symbol Transistor_FET:IRLZ44N
- added R10, R8, R9: R, Resistor_SMD:R_0805_2012Metric, symbol Device:R
- C1, C4: footprint (none) -> Capacitor_SMD:C_0805_2012Metric
- C2: footprint (none) -> Capacitor_THT:CP_Radial_D5.0mm_P2.00mm
- C3, C6, C8: footprint (none) -> Capacitor_SMD:CP_Elec_8x5.4
- D1, D2, D3, D4, D5: footprint (none) -> LED_SMD:LED_0805_2012Metric
- D12, D13, D7, D8, D9: footprint (none) -> Diode_SMD:D_0805_2012Metric
- D6: footprint (none) -> OptoDevice:Osram_BPW34S-SMD
- J5, J6: footprint (none) -> TerminalBlock_Phoenix:TerminalBlock_Phoenix_PTSM-0,5-2-2,5-V-SMD_1x02-1MP_P2.50mm_Vertical
- L1: footprint (none) -> Inductor_SMD:L_Neosid_Ms85
- R1, R2, R5, R6, R7: footprint (none) -> Resistor_SMD:R_0805_2012Metric
- RV1: footprint (none) -> Potentiometer_SMD:Potentiometer_ACP_CA6-VSMD_Vertical
Connections:
- net +5V: now also C3.1, C4.1, L1.2, R6.1, RV1.3, J2.15 (Pin_15), J8.1 (Pin_1), Q1.1 (G); no longer U1.11 (EnB)
- net IN1: now also J7.7 (Pin_7)
- net IN2: now also J7.10 (Pin_10)
- net OUT1: now also J1.1 (Pin_1)
- net OUT2: now also J1.2 (Pin_2)
- net VBAT: now also C1.1, C2.1, U4.1 (VIN); no longer J5.3 (Pin_3)
- net at R2.1: now also D2.2 (A)
- net -BATT: now reaches R2.2
- net -BATT: now also C1.2, C2.2, C3.2, C4.2, C6.2, C8.2, D12.1 (K), D13.1 (K), D3.2 (A), D4.2 (A), D5.1 (K), D6.1 (K), D7.2 (A), J5.3 (Pin_3), R1.2, R7.2, U1.1 (SENSE_A), U1.8 (GND), U2.2 (GND), U4.3 (GND), U4.5 (~{ON}/OFF), J7.20 (Pin_20), J8.2 (Pin_2), Q1.3 (S)
- net Q1: now reaches D1.1 (K)
- net Q1: now also R8.2
- net at D1.2 (A): now also R1.1
- net Q3: now reaches D4.1 (K)
- net Q3: now also D3.1 (K), R10.1
- net Q2: now reaches D2.1 (K)
- net Q2: now also R9.2
- removed net GND: C1.2, C2.2, C3.2, C4.2, C6.2, C8.2, D12.1 (K), D13.1 (K), D5.1 (K), D6.1 (K), D7.2 (A), J5.2 (Pin_2), R7.2, U1.1 (SENSE_A), U1.15 (SENSE_B), U1.8 (GND), U2.2 (GND), U4.3 (GND), U4.5 (~{ON}/OFF)
- net IN3: no longer names the net of U1.10 (IN3)
- net IN4: no longer names the net of U1.12 (IN4)
- new net: Q1.2 (D), R10.2
- new net: J7.16 (Pin_16), R8.1
- new net: J7.15 (Pin_15), R9.1
- new net +BATT: J5.2 (Pin_2)
- new net servosignal: J7.6 (Pin_6), J8.3 (Pin_3)
- no-connect marks 0 -> 39
Other:
- note added: "LOLIN32"
- note added: "MOSFET"
- note added: "Prednja svjetla + pokazivači smjera"
- note added: "Servo motor + motor"
- moved on the sheet: D1, D12, D13, D2, D3, D4, D8, D9, J6, R1, R2
