File: Tiskana_plocica_za_lego_auto/Tiskana_plocica_za_lego_auto.kicad_sch (KiCad schematic)
At the start: 41 parts, among them J1 Conn_01x02_Socket, J2 Conn_01x20_Socket, J6 Screw_Terminal_01x02, J7 Conn_01x20_Socket, J8 Conn_01x03_Pin, Q1 IRLZ44N, U1 L298N, U2 LM78M05_TO220, U4 LM2596S-5

Commit message: pcb
Parts:
- J5: footprint TerminalBlock_Phoenix:TerminalBlock_Phoenix_PTSM-0,5-2-2,5-V-SMD_1x02-1MP_P2.50mm_Vertical -> TerminalBlock_Phoenix:TerminalBlock_Phoenix_PTSM-0,5-3-2,5-V-SMD_1x03-1MP_P2.50mm_Vertical
Changed lines of the file:
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@@
 			)
 		)
-		(property "Footprint" "TerminalBlock_Phoenix:TerminalBlock_Phoenix_PTSM-0,5-2-2,5-V-SMD_1x02-1MP_P2.50mm_Vertical"
+		(property "Footprint" "TerminalBlock_Phoenix:TerminalBlock_Phoenix_PTSM-0,5-3-2,5-V-SMD_1x03-1MP_P2.50mm_Vertical"
 			(at 19.05 69.85 0)
 			(effects

Commit message: fix2
Parts:
- C1: Manufacturer (none) -> muRata; ManufacturersPartNumber (none) -> GRM31C5C1H104JA01L
- C2: Manufacturer (none) -> VISHAY; ManufacturersPartNumber (none) -> 293D107X9010C2TE3
- J2: footprint Connector_PinHeader_2.54mm:PinHeader_1x20_P2.54mm_Vertical_SMD_Pin1Left -> Connector_PinSocket_2.54mm:PinSocket_1x20_P2.54mm_Vertical_SMD_Pin1Right
Changed lines of the file:
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@@
+			)
+		)
+		(property "Manufacturer" "  VISHAY "
+			(at 41.91 41.91 0)
+			(effects
+				(font
+					(size 1.27 1.27)
+				)
+				(hide yes)
+			)
+		)
+		(property "ManufacturersPartNumber" "293D107X9010C2TE3"
+			(at 41.91 41.91 0)
+			(effects
+				(font
+					(size 1.27 1.27)
+				)
+				(hide yes)
 			)
 		)
@@
 			)
 		)
+		(property "Manufacturer" "  muRata "
+			(at 49.53 41.91 0)
+			(effects
+				(font
+					(size 1.27 1.27)
+				)
+				(hide yes)
+			)
+		)
+		(property "ManufacturersPartNumber" "GRM31C5C1H104JA01L"
+			(at 49.53 41.91 0)
+			(effects
+				(font
+					(size 1.27 1.27)
+				)
+				(hide yes)
+			)
+		)
 		(pin "2"
 		)
@@
 			)
 		)
-		(property "Footprint" "Connector_PinHeader_2.54mm:PinHeader_1x20_P2.54mm_Vertical_SMD_Pin1Left"
+		(property "Footprint" "Connector_PinSocket_2.54mm:PinSocket_1x20_P2.54mm_Vertical_SMD_Pin1Right"
 			(at 203.2 105.41 0)
 			(effects
