File: Tiskana_plocica_za_lego_auto/Tiskana_plocica_za_lego_auto.kicad_pcb (KiCad board)
At the start: 2 copper layers, 140 x 100 mm, 41 parts, among them J1 Conn_01x02_Socket, J2 Conn_01x20_Socket, J6 Screw_Terminal_01x02, J7 Conn_01x20_Socket, J8 Conn_01x03_Pin, Q1 IRLZ44N, U1 L298N, U2 LM78M05_TO220, U4 LM2596S-5

Commit message: pcb
Parts:
- moved J1 0.34 mm to (131.0, 88.7)
Routing:
- net -BATT: track 0.00 -> 331.6 mm, vias 0 -> 28
- net +5V: track 0.00 -> 226.2 mm, vias 0 -> 4
- net Net-(J7-Pin_16): track 0.00 -> 142.7 mm, vias 0 -> 2
- net VBAT: track 0.00 -> 130.5 mm, vias 0 -> 2
- net Net-(J7-Pin_15): track 0.00 -> 128.3 mm, vias 0 -> 2
- net /IN2: track 0.00 -> 91.3 mm, vias 0 -> 2
- net /servosignal: track 0.00 -> 84.1 mm, vias 0 -> 4
- net /IN1: track 0.00 -> 63.2 mm
- net /FB R4: track 0.00 -> 51.0 mm, vias 0 -> 2
- net Net-(D13-A): track 0.00 -> 46.1 mm, vias 0 -> 2
- net Q3: track 0.00 -> 42.0 mm
- net Net-(D12-A): track 0.00 -> 40.3 mm, vias 0 -> 4
- net Net-(D7-K): track 0.00 -> 30.2 mm, vias 0 -> 2
- net /OUT1: track 0.00 -> 28.3 mm
- net Q1: track 0.00 -> 19.7 mm
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
Commit message: fix2
Parts:
- J2: footprint Connector_PinHeader_2.54mm:PinHeader_1x20_P2.54mm_Vertical_SMD_Pin1Left -> Connector_PinSocket_2.54mm:PinSocket_1x20_P2.54mm_Vertical_SMD_Pin1Right
